File: hardware/MDR_50Pin/MDR_50Pin.kicad_sch (KiCad schematic)
At the start: 65 parts, among them J2 TRM_BCKF, Q3 AO3401A, U10 Centronics50PinMale, U3 AP1117-ADJ, U4 LVTH245, U5 LVT125, U6 LVT125, U7 LVT125, U9 LVTH245

Commit message: latest design
Parts:
- removed C16: 10uF, Capacitor_SMD:C_0603_1608Metric, symbol Device:CP
- removed D4: D, Diode_SMD:D_SMA, symbol Device:D
- removed F1: Polyfuse, Fuse:Fuse_0805_2012Metric_Pad1.15x1.40mm_HandSolder, symbol Device:Polyfuse
- removed J2: TRM_BCKF, Connector_PinHeader_2.54mm:PinHeader_1x02_P2.54mm_Vertical, symbol Connector:Conn_01x02_Pin
- removed Q3: AO3401A, Package_TO_SOT_SMD:SOT-23, symbol Transistor_FET:AO3401A
- removed R11: 10k, Resistor_SMD:R_0603_1608Metric, symbol Device:R
- removed R20: 154, Resistor_SMD:R_0603_1608Metric, symbol Device:R
- removed R21: 120, Resistor_SMD:R_0805_2012Metric, symbol Device:R
- C1, C11, C13, C14, C2, C5, C8, C9: LCSC Part # (none) -> C14663
- C10, C12, C15, C6: LCSC Part # (none) -> C19666
- C3: footprint Capacitor_SMD:C_1206_3216Metric_Pad1.42x1.75mm_HandSolder -> Capacitor_SMD:C_1206_3216Metric; LCSC Part # (none) -> C5672
- C4: footprint Capacitor_SMD:C_1206_3216Metric_Pad1.42x1.75mm_HandSolder -> Capacitor_SMD:C_1206_3216Metric; LCSC Part # (none) -> C96123
- D1: LCSC Part # (none) -> C2480
- F2: footprint Fuse:Fuse_0805_2012Metric_Pad1.15x1.40mm_HandSolder -> Fuse:Fuse_0805_2012Metric; LCSC Part # (none) -> C883111
- R1, R10, R2, R3, R33, R34, R35, R36, R37, R38, R39, R4, R40, R5, R6, R7, R8, R9: footprint Resistor_SMD:R_0603_1608Metric_Pad0.98x0.95mm_HandSolder -> Resistor_SMD:R_0402_1005Metric; LCSC Part # (none) -> C25078
- R12, R13, R14, R15, R16, R17, R18, R19, R42: footprint Resistor_SMD:R_0402_1005Metric_Pad0.72x0.64mm_HandSolder -> Resistor_SMD:R_0402_1005Metric; LCSC Part # (none) -> C11702
- R22, R23, R25: footprint Resistor_SMD:R_0603_1608Metric_Pad0.98x0.95mm_HandSolder -> Resistor_SMD:R_0402_1005Metric; LCSC Part # (none) -> C25900
- R28, R29: footprint Resistor_SMD:R_0603_1608Metric_Pad0.98x0.95mm_HandSolder -> Resistor_SMD:R_0402_1005Metric; LCSC Part # (none) -> C11702
- RP1: footprint CustomFootprints:BluePillModule -> Library:RPi_Pico_SMD; now left out of the parts list
- SD2: footprint Library:TF-06_MicroSD -> Library:TF-SMD_TF-06A; LCSC Part # (none) -> C693844
- U10: value Centronics50PinMale -> MDR50; footprint Library:Centronics50Male -> Library:MDR50; now left out of the parts list
- U3: value AP1117-ADJ -> AMS1117-2.85; LCSC Part # (none) -> C14791
- U4, U9: LCSC Part # (none) -> C2652121
- U5, U6, U7: LCSC Part # (none) -> C7042
Connections:
- net GND: now also U3.1 (ADJ)
Other:
- note added: "(Adjustable: Stuff R20, R21, and C16 as shown) Fixed: Omit R21 and C16, swap R20 to 0 ohm jumper"
- note removed: "Adjustable: Stuff R20, R21, and C16 as shown Fixed: Omit R21 and C16, swap R20 to 0 ohm jumper"
